File: Hardware/Servo.sch (EAGLE design)
At the start: 15 parts, among them T1 BC337, T2 BC337, U1 PIC16F1508-I/P

Commit message: 1/12
Parts:
- removed R5, R6: (no value), rcl:R-US_R0603
- removed T1, T2: BC337, transistor:BC337
- removed U1: PIC16F1508-I/P, pic16f1508:PIC16F1508-I/P
- added IC1: PIC16F1508, ic-package:DIL20S
- added R2, R3: 3.3k, rcl:R-US_V526-0
- added T3, T4: 2SC1815, transistor:2SC1815
- C1: value (none) -> 4.7uF
- C2: value (none) -> 100uF
- CN1: value (none) -> ICSP
- CN3: value (none) -> Servo1
- CN4: value (none) -> Servo2
- JP1: value (none) -> Raspi
- R1: value (none) -> 10k; device rcl:R-US_R0603 -> rcl:R-US_V526-0
- R4, R7: value (none) -> 5.1k; device rcl:R-US_R0603 -> rcl:R-US_V526-0
- SW1: value (none) -> Reset
Connections:
- removed net N$10: JP1.10, U1.RB5/AN11/CLC4IN0/RX/DT
- removed net N$16: R6.2, U1.RC0/AN4/CLC2/C2IN+
- removed net N$17: R5.1, T1.B
- removed net N$18: R6.1, T2.B
- removed net N$24: CN3.1, R4.2, T1.C
- new net N$12: IC1.16, R3.2
- new net N$13: R2.1, T3.B
- new net N$14: R3.1, T4.B
- new net N$6: IC1.11, JP1.8
- new net N$7: IC1.12, JP1.10
- net GND1: now also IC1.20, T3.E, T4.E; no longer T1.E, T2.E, U1.VSS
- net N$1: now also IC1.10; no longer U1.RB7/CLC3/TX/CK
- net N$11: now also IC1.17, R2.2; no longer JP1.12, U1.RB4/AN10/CLC3IN0/SDA/SDI
- net N$15: now also CN3.1, R4.2, T3.C; no longer R5.2, U1.RA2/AN2/C1OUT/DAC1OUT2/T0CKI/INT/PWM3/CLC1/!CWG1FLT
- net N$19: now also CN1.4, IC1.19; no longer CN1.5, U1.RA1/AN1/CLC4IN1/VREF+/C1IN0-/C2IN0-/ICSPCLK/ICDCLK
- net N$2: now also IC1.9; no longer U1.RC7/AN9/CLC1IN1/SDO
- net N$20: now also CN1.5, IC1.18; no longer CN1.4, U1.RA0/AN0/C1IN+/DAC1OUT1/ICSPDAT/ICDDAT
- net N$3: now also IC1.8; no longer U1.RC6/AN8/NCO1/CLC3IN1/!SS
- net N$4: now also T4.C; no longer T2.C
- net N$5: now also IC1.7; no longer U1.RC3/AN7/C1IN3-/C2IN3-/PWM2/CLC2IN0
- net N$8: now also IC1.4; no longer U1.RA3/CLC1IN0/VPP/T1G/!SS/!MCLR
- net N$9: now also IC1.13, JP1.12; no longer JP1.8, U1.RB6/SCL/SCK
- net VDD: now also IC1.1; no longer U1.VDD
Other:
- moved on the sheet: C1, C2, CN3, CN4, R4, R7
